File: KiCad_new/att_10db/att_10db.kicad_pcb (KiCad board)
At the start: 2 copper layers, 6 parts

Commit message: One more GND pad dded
Parts:
- added Gnd2: MountingHole_Pad, TestPoint:TestPoint_Pad_2.5x2.5mm, F.Cu at (147.3, 102.9)
Connections:
- R2 pad 1: Net-(Out1-Pad1) -> Net-(In1-Pad1)
- R2 pad 2: Net-(In1-Pad1) -> Net-(Out1-Pad1)
Changed lines of the file:
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@@
     (tracks 18)
     (zones 0)
-    (modules 6)
+    (modules 7)
     (nets 4)
   )
@@
   )
   (setup
-    (last_trace_width 2)
+    (last_trace_width 0.25)
     (user_trace_width 2)
     (trace_clearance 0.2)
@@
   )
   (module TestPoint:TestPoint_Pad_2.5x2.5mm (layer F.Cu)
+    (at 147.32 102.87)
+    (descr "SMD rectangular pad as test Point, square 2.5mm side length")
+    (tags "test point SMD pad rectangle square")
+    (attr virtual)
+    (fp_text reference Gnd2 (at 0 -2.148) (layer F.SilkS)
+      (effects (font (size 1 1) (thickness 0.15)))
+    )
+    (fp_text value MountingHole_Pad (at 0 2.25) (layer F.Fab)
+      (effects (font (size 1 1) (thickness 0.15)))
+    )
+    (fp_line (start 1.75 1.75) (end -1.75 1.75) (layer F.CrtYd) (width 0.05))
+    (fp_line (start 1.75 1.75) (end 1.75 -1.75) (layer F.CrtYd) (width 0.05))
+    (fp_line (start -1.75 -1.75) (end -1.75 1.75) (layer F.CrtYd) (width 0.05))
+    (fp_line (start -1.75 -1.75) (end 1.75 -1.75) (layer F.CrtYd) (width 0.05))
+    (fp_line (start -1.45 1.45) (end -1.45 -1.45) (layer F.SilkS) (width 0.12))
+    (fp_line (start 1.45 1.45) (end -1.45 1.45) (layer F.SilkS) (width 0.12))
+    (fp_line (start 1.45 -1.45) (end 1.45 1.45) (layer F.SilkS) (width 0.12))
+    (fp_line (start -1.45 -1.45) (end 1.45 -1.45) (layer F.SilkS) (width 0.12))
+    (fp_text user %R (at 0 -2.15) (layer F.Fab)
+      (effects (font (size 1 1) (thickness 0.15)))
+    )
+    (pad 1 smd rect (at 0 0) (size 2.5 2.5) (layers F.Cu F.Mask)
+      (net 1 GNDREF))
+  )
+  (module TestPoint:TestPoint_Pad_2.5x2.5mm (layer F.Cu)
     (at 124.46 102.87)
     (descr "SMD rectangular pad as test Point, square 2.5mm side length")
@@
     (fp_circle (center 2.54 -16.66) (end 4.39 -16.66) (layer F.Fab) (width 0.1))
     (pad 2 thru_hole oval (at 5.08 0 180) (size 2 2) (drill 1.1) (layers *.Cu *.Mask)
+      (net 3 "Net-(Out1-Pad1)"))
+    (pad 1 thru_hole rect (at 0 0 180) (size 2 2) (drill 1.1) (layers *.Cu *.Mask)
       (net 2 "Net-(In1-Pad1)"))
-    (pad 1 thru_hole rect (at 0 0 180) (size 2 2) (drill 1.1) (layers *.Cu *.Mask)
-      (net 3 "Net-(Out1-Pad1)"))
     (pad "" np_thru_hole oval (at 2.54 -16.66 180) (size 3.5 3.5) (drill 3.5) (layers *.Cu *.Mask))
     (model ${KISYS3DMOD}/Package_TO_SOT_THT.3dshapes/TO-220-2_Horizontal_TabDown.wrl
